File: pcb/Ultrasonic_mux.sch (KiCad schematic (older format))
At the start: 70 parts, among them J0 DB9_Male, J1 DB9_Male, J10 Conn_01x03_Male, J11 Conn_01x03_Male, J12 Conn_01x03_Male, J13 Conn_01x03_Male, J14 Conn_01x03_Male, J15 Conn_01x03_Male, J2 DB9_Male, J3 DB9_Male, J4 DB9_Male, J5 DB9_Male, P1 , P12 , P27 , P28 , P3 , P5 , Q0 MMBT3904, Q1 MMBT3904, Q2 MMBT3904, Q3 MMBT3904, Q4 MMBT3904, Q5 MMBT3904, U1 FeatherM0

Commit message: Hopefully finished track routes.
Parts:
- +3V3p1, +5Vp1, GNDp1: footprint Pin_Headers:Pin_Header_Angled_1x01_Pitch2.54mm -> Pin_Headers:Pin_Header_Straight_1x01_Pitch2.54mm
Changed lines of the file:
@@
 F 0 "+5Vp1" V 6850 2400 50  0000 C CNN
 F 1 " " H 6750 2300 50  0000 C CNN
-F 2 "Pin_Headers:Pin_Header_Angled_1x01_Pitch2.54mm" H 6750 2400 50  0001 C CNN
+F 2 "Pin_Headers:Pin_Header_Straight_1x01_Pitch2.54mm" H 6750 2400 50  0001 C CNN
 F 3 "" H 6750 2400 50  0001 C CNN
 	1    6750 2400
@@
 F 0 "+3V3p1" V 7200 2450 50  0000 C CNN
 F 1 " " H 7100 2350 50  0000 C CNN
-F 2 "Pin_Headers:Pin_Header_Angled_1x01_Pitch2.54mm" H 7100 2450 50  0001 C CNN
+F 2 "Pin_Headers:Pin_Header_Straight_1x01_Pitch2.54mm" H 7100 2450 50  0001 C CNN
 F 3 "" H 7100 2450 50  0001 C CNN
 	1    7100 2450
@@
 F 0 "GNDp1" V 7550 2200 50  0000 C CNN
 F 1 " " H 7450 2100 50  0000 C CNN
-F 2 "Pin_Headers:Pin_Header_Angled_1x01_Pitch2.54mm" H 7450 2200 50  0001 C CNN
+F 2 "Pin_Headers:Pin_Header_Straight_1x01_Pitch2.54mm" H 7450 2200 50  0001 C CNN
 F 3 "" H 7450 2200 50  0001 C CNN
 	1    7450 2200
